Commit message: Add

File: jedy/jedy_description/urdf/jedy_four_dof_with_yaw.urdf (robot description, URDF)
Before this commit: robot test_robot, 39 links, 38 joints
Links:
- link base_link: geometry collision mesh filename=package://jedy_description/meshes/screw_body_module/base_li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; visual mesh filename=package://jedy_description/meshes/screw_body_module/base_li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
- link head_link0: geometry collision mesh filename=package://jedy_description/meshes/screw_body_module/head_li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; visual mesh filename=package://jedy_description/meshes/screw_body_module/head_li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
- link head_module1_base_link: geometry collision mesh filename=package://jedy_description/meshes/screw_20mmhead_module_cov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; visual mesh filename=package://jedy_description/meshes/screw_20mmhead_module_cov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
- link head_module1_link1: geometry collision mesh filename=package://jedy_description/meshes/screw_20mmhead_module_cov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; visual mesh filename=package://jedy_description/meshes/screw_20mmhead_module_cov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
- link larm_link0: geometry collision mesh filename=package://jedy_description/meshes/screw_body_module/larm_li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; visual mesh filename=package://jedy_description/meshes/screw_body_module/larm_li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
- link larm_module1_base_link: geometry collision mesh filename=package://jedy_description/meshes/screw_crosscantileverleft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; visual mesh filename=package://jedy_description/meshes/screw_crosscantileverleft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
- link larm_module1_link1: geometry collision mesh filename=package://jedy_description/meshes/screw_crosscantileverleft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; visual mesh filename=package://jedy_description/meshes/screw_crosscantileverleft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
- link larm_module1_link2: geometry collision mesh filename=package://jedy_description/meshes/screw_crosscantileverleft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; visual mesh filename=package://jedy_description/meshes/screw_crosscantileverleft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
- link larm_module2_base_link: geometry collision mesh filename=package://jedy_description/meshes/screw_26mmhinge_module_co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; visual mesh filename=package://jedy_description/meshes/screw_26mmhinge_module_co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
- link larm_module2_link1: geometry collision mesh filename=package://jedy_description/meshes/screw_26mmhinge_module_co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; visual mesh filename=package://jedy_description/meshes/screw_26mmhinge_module_co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
- link larm_module3_base_link: geometry collision mesh filename=package://jedy_description/meshes/screw_yaw_module/base_lin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; visual mesh filename=package://jedy_description/meshes/screw_yaw_module/base_lin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
- link larm_module3_dummy_link: geometry collision mesh filename=package://jedy_description/meshes/screw_yaw_module/dummy_li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; visual mesh filename=package://jedy_description/meshes/screw_yaw_module/dummy_li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
- link larm_module3_link1: geometry collision mesh filename=package://jedy_description/meshes/screw_yaw_module/link1.dae; visual mesh filename=package://jedy_description/meshes/screw_yaw_module/link1.dae
- link left_hand_base_link: geometry collision mesh filename=package://jedy_description/meshes/screw_hand_module/base_li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; visual mesh filename=package://jedy_description/meshes/screw_hand_module/base_li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
- link left_hand_link1: geometry collision mesh filename=package://jedy_description/meshes/screw_hand_module/link1.d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; visual mesh filename=package://jedy_description/meshes/screw_hand_module/link1.d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
- link left_hand_link2: geometry collision mesh filename=package://jedy_description/meshes/screw_hand_module/link2.d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; visual mesh filename=package://jedy_description/meshes/screw_hand_module/link2.d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
- link mechanum_base_link: geometry collision mesh filename=package://jedy_description/meshes/screw_mechanum_module/bas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; visual mesh filename=package://jedy_description/meshes/screw_mechanum_module/bas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
- link mechanum_link1: geometry collision mesh filename=package://jedy_description/meshes/screw_mechanum_module/lin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; visual mesh filename=package://jedy_description/meshes/screw_mechanum_module/lin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
- link mechanum_link2: geometry collision mesh filename=package://jedy_description/meshes/screw_mechanum_module/lin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; visual mesh filename=package://jedy_description/meshes/screw_mechanum_module/lin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
- link mechanum_link3: geometry collision mesh filename=package://jedy_description/meshes/screw_mechanum_module/lin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; visual mesh filename=package://jedy_description/meshes/screw_mechanum_module/lin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
- link mechanum_link4: geometry collision mesh filename=package://jedy_description/meshes/screw_mechanum_module/lin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; visual mesh filename=package://jedy_description/meshes/screw_mechanum_module/lin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
- link rarm_link0: geometry collision mesh filename=package://jedy_description/meshes/screw_body_module/rarm_li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; visual mesh filename=package://jedy_description/meshes/screw_body_module/rarm_li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
- link rarm_module1_base_link: geometry collision mesh filename=package://jedy_description/meshes/screw_crosscantileverrigh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; visual mesh filename=package://jedy_description/meshes/screw_crosscantileverrigh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
- link rarm_module1_link1: geometry collision mesh filename=package://jedy_description/meshes/screw_crosscantileverrigh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; visual mesh filename=package://jedy_description/meshes/screw_crosscantileverrigh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
- link rarm_module1_link2: geometry collision mesh filename=package://jedy_description/meshes/screw_crosscantileverrigh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; visual mesh filename=package://jedy_description/meshes/screw_crosscantileverrigh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
- link rarm_module2_base_link: geometry collision mesh filename=package://jedy_description/meshes/screw_26mmhinge_module_co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; visual mesh filename=package://jedy_description/meshes/screw_26mmhinge_module_co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
- link rarm_module2_link1: geometry collision mesh filename=package://jedy_description/meshes/screw_26mmhinge_module_co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; visual mesh filename=package://jedy_description/meshes/screw_26mmhinge_module_co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
- link right_hand_base_link: geometry collision mesh filename=package://jedy_description/meshes/screw_hand_module/base_li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; visual mesh filename=package://jedy_description/meshes/screw_hand_module/base_li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
- link right_hand_link1: geometry collision mesh filename=package://jedy_description/meshes/screw_hand_module/link1.d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; visual mesh filename=package://jedy_description/meshes/screw_hand_module/link1.d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
- link right_hand_link2: geometry collision mesh filename=package://jedy_description/meshes/screw_hand_module/link2.d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; visual mesh filename=package://jedy_description/meshes/screw_hand_module/link2.d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
Joints:
- joint dummy_joint_head: limit lower=-1.57 upper=1.57 effort=0.48 velocity=6.55 -> lower=-1.57 upper=1.57 effort=0.48 velocity=7.4
- joint dummy_joint_larm: limit lower=-0.56 upper=2.35 effort=0.48 velocity=6.55 -> lower=-0.56 upper=2.35 effort=0.48 velocity=7.4
- joint dummy_joint_lleg: limit effort=0.48 velocity=6.55 -> effort=0.48 velocity=7.4
- joint dummy_joint_rarm: limit lower=-2.35 upper=0.52 effort=0.48 velocity=6.55 -> lower=-2.35 upper=0.52 effort=0.48 velocity=7.4
- joint dummy_joint_rleg: limit effort=0.48 velocity=6.55 -> effort=0.48 velocity=7.4
- joint head_joint0: limit lower=-2.35 upper=2.35 effort=0.48 velocity=6.55 -> lower=-2.35 upper=2.35 effort=0.48 velocity=7.4
- joint head_module1_base_link_to_dummy_link_head_joint: axis (none) -> 1. 0. 0.; limit (none) -> effort=0.0 velocity=0.0; origin xyz=0 0 0 rpy=0 0 0 -> xyz=0.0 0.0 0.0 rpy=0.0 -0.0 0.0
- joint head_module1_joint1: limit lower=-1.57 upper=1.57 effort=0.0 velocity=0.0 -> lower=-1.57 upper=1.57 effort=0.0 velocity=7.4
- joint larm_joint0: limit lower=-2.35 upper=2.35 effort=0.48 velocity=6.55 -> lower=-2.35 upper=2.35 effort=0.48 velocity=7.4
- joint larm_module1_base_link_to_dummy_link_larm_joint: axis (none) -> 1. 0. 0.; limit (none) -> effort=0.0 velocity=0.0; origin xyz=0 0 0 rpy=0 0 -1.5707963267948966 -> xyz=0.0 0.0 0.0 rpy=-0.0 -0.0 -1.5707963267948963
- joint larm_module1_joint1: limit lower=-1.57 upper=0.087 effort=0.0 velocity=0.0 -> lower=-1.57 upper=0.087 effort=0.0 velocity=7.4
- joint larm_module1_joint2: limit lower=-2.35 upper=2.35 effort=0.0 velocity=0.0 -> lower=-2.35 upper=2.35 effort=0.0 velocity=7.4
- joint larm_module2_base_link_to_larm_module1_dummy_link_joint: axis (none) -> 1. 0. 0.; limit (none) -> effort=0.0 velocity=0.0; origin xyz=0 0 0 rpy=0 0 0 -> xyz=0.0 0.0 0.0 rpy=0.0 -0.0 0.0
- joint larm_module2_joint1: limit lower=-1.78 upper=1.78 effort=0.0 velocity=0.0 -> lower=-1.78 upper=1.78 effort=0.0 velocity=7.4
- joint larm_module3_base_link_to_larm_module2_dummy_link_joint: axis (none) -> 1. 0. 0.; limit (none) -> effort=0.0 velocity=0.0; origin xyz=0 0 0 rpy=0 0 0 -> xyz=0.0 0.0 0.0 rpy=0.0 -0.0 0.0
- joint larm_module3_joint1: limit lower=-2.356 upper=2.356 effort=0.0 velocity=7.0 -> lower=-2.356 upper=2.356 effort=0.0 velocity=7.4
- joint left_hand_base_link_to_larm_module3_dummy_link_joint: axis (none) -> 1. 0. 0.; limit (none) -> effort=0.0 velocity=0.0; origin xyz=0 0 0 rpy=0 0 0 -> xyz=0.0 0.0 0.0 rpy=0.0 -0.0 0.0
- joint left_hand_joint1: limit lower=-0.43 upper=1.57 effort=0.0 velocity=0.0 -> lower=-0.43 upper=1.57 effort=0.0 velocity=7.4
- joint left_hand_joint2: limit lower=-0.43 upper=1.57 effort=0.0 velocity=0.0 -> lower=-0.43 upper=1.57 effort=0.0 velocity=7.4
- joint mechanum_base_link_to_dummy_link_rleg_joint: axis (none) -> 1. 0. 0.; limit (none) -> effort=0.0 velocity=0.0; origin xyz=0 0 0 rpy=0 0 0 -> xyz=0.0 0.0 0.0 rpy=0.0 -0.0 0.0
- joint mechanum_joint1: limit effort=0.48 velocity=6.55 -> effort=0.48 velocity=7.4
- joint mechanum_joint2: limit effort=0.48 velocity=6.55 -> effort=0.48 velocity=7.4
- joint mechanum_joint3: limit effort=0.48 velocity=6.55 -> effort=0.48 velocity=7.4
- joint mechanum_joint4: limit effort=0.48 velocity=6.55 -> effort=0.48 velocity=7.4
- joint rarm_joint0: limit lower=-2.35 upper=2.35 effort=0.48 velocity=6.55 -> lower=-2.35 upper=2.35 effort=0.48 velocity=7.4
- joint rarm_module1_base_link_to_dummy_link_rarm_joint: axis (none) -> 1. 0. 0.; limit (none) -> effort=0.0 velocity=0.0; origin xyz=0 0 0 rpy=0 0 -1.5707963267948966 -> xyz=0.0 0.0 0.0 rpy=-0.0 -0.0 -1.5707963267948963
- joint rarm_module1_joint1: limit lower=-1.57 upper=0.087 effort=0.0 velocity=0.0 -> lower=-1.57 upper=0.087 effort=0.0 velocity=7.4
- joint rarm_module1_joint2: limit lower=-2.35 upper=2.35 effort=0.0 velocity=0.0 -> lower=-2.35 upper=2.35 effort=0.0 velocity=7.4
- joint rarm_module2_base_link_to_rarm_module1_dummy_link_joint: axis (none) -> 1. 0. 0.; limit (none) -> effort=0.0 velocity=0.0; origin xyz=0 0 0 rpy=0 0 0 -> xyz=0.0 0.0 0.0 rpy=0.0 -0.0 0.0
- joint rarm_module2_joint1: limit lower=-1.78 upper=1.78 effort=0.0 velocity=0.0 -> lower=-1.78 upper=1.78 effort=0.0 velocity=7.4
- joint right_hand_base_link_to_rarm_module2_dummy_link_joint: axis (none) -> 1. 0. 0.; limit (none) -> effort=0.0 velocity=0.0; origin xyz=0 0 0 rpy=0 0 0 -> xyz=0.0 0.0 0.0 rpy=0.0 -0.0 0.0
- joint right_hand_joint1: limit lower=-0.43 upper=1.57 effort=0.0 velocity=0.0 -> lower=-0.43 upper=1.57 effort=0.0 velocity=7.4
- joint right_hand_joint2: limit lower=-0.43 upper=1.57 effort=0.0 velocity=0.0 -> lower=-0.43 upper=1.57 effort=0.0 velocity=7.4

Commit message: Add

File: jedy/jedy_description/urdf/jedy_four_dof_with_yaw.urdf (robot description, URDF)
Before this commit: robot test_robot, 39 links, 38 joints
Joints:
- joint larm_module3_base_link_to_larm_module2_dummy_link_joint: origin xyz=0.0 0.0 0.0 rpy=0.0 -0.0 0.0 -> xyz=0.0 0.0 0.0 rpy=0.0 -0.0 3.14
