Commit message: Add

File: jedy/jedy_description/urdf/jedy_no_arm.urdf (robot description, URDF)
Before this commit: robot jedy, 14 links, 13 joints
Links:
- link camera_link: geometry visual box size=0.01 0.01 0.01

Commit message: Add

File: jedy/jedy_description/urdf/jedy_no_arm.urdf (robot description, URDF)
Before this commit: robot jedy, 14 links, 13 joints
Links:
- link camera_link: geometry collision box size=0.01 0.01 0.01; visual box size=0.01 0.01 0.01
