Commit message: Add

File: jedy/jedy_description/urdf/jedy_four_dof.urdf (robot description, URDF)
Before this commit: robot test_robot, 36 links, 35 joints
Links:
- link mechanum_base_link: geometry collision cylinder length=0.02 radius=0.03; visual mesh filename=package://screw_mechanum_module/meshes/base_link.dae
- link mechanum_link1: geometry collision cylinder length=0.02 radius=0.03; visual mesh filename=package://screw_mechanum_module/meshes/link1.dae
- link mechanum_link2: geometry collision cylinder length=0.02 radius=0.03; visual mesh filename=package://screw_mechanum_module/meshes/link2.dae
- link mechanum_link3: geometry collision cylinder length=0.02 radius=0.03; visual mesh filename=package://screw_mechanum_module/meshes/link3.dae
- link mechanum_link4: geometry collision cylinder length=0.02 radius=0.03; visual mesh filename=package://screw_mechanum_module/meshes/link4.dae

Commit message: Add

File: jedy/jedy_description/urdf/jedy_four_dof.urdf (robot description, URDF)
Before this commit: robot test_robot, 36 links, 35 joints
Joints:
- joint larm_module1_joint1: limit lower=-1.57 upper=0.087 effort=0.0 velocity=0.0 -> lower=-1.57 upper=0.087 effort=0.0 velocity=6.5
- joint larm_module1_joint2: limit lower=-2.35 upper=2.35 effort=0.0 velocity=0.0 -> lower=-2.35 upper=2.35 effort=0.0 velocity=6.5
- joint larm_module2_joint1: limit lower=-1.78 upper=1.78 effort=0.0 velocity=0.0 -> lower=-1.78 upper=1.78 effort=0.0 velocity=6.5
- joint left_hand_joint1: limit lower=-0.43 upper=1.57 effort=0.0 velocity=0.0 -> lower=-0.43 upper=1.57 effort=0.0 velocity=6.5
- joint left_hand_joint2: limit lower=-0.43 upper=1.57 effort=0.0 velocity=0.0 -> lower=-0.43 upper=1.57 effort=0.0 velocity=6.5
- joint rarm_module1_joint1: limit lower=-1.57 upper=0.087 effort=0.0 velocity=0.0 -> lower=-1.57 upper=0.087 effort=0.0 velocity=6.5
- joint rarm_module1_joint2: limit lower=-2.35 upper=2.35 effort=0.0 velocity=0.0 -> lower=-2.35 upper=2.35 effort=0.0 velocity=6.5
- joint right_hand_joint1: limit lower=-0.43 upper=1.57 effort=0.0 velocity=0.0 -> lower=-0.43 upper=1.57 effort=0.0 velocity=6.5
- joint right_hand_joint2: limit lower=-0.43 upper=1.57 effort=0.0 velocity=0.0 -> lower=-0.43 upper=1.57 effort=0.0 velocity=6.5

Commit message: Add

File: jedy/jedy_description/urdf/jedy_four_dof.urdf (robot description, URDF)
Before this commit: robot test_robot, 36 links, 35 joints
Joints:
- joint head_module1_joint1: limit lower=-1.57 upper=1.57 effort=0.0 velocity=0.0 -> lower=-1.57 upper=1.57 effort=0.0 velocity=6.5
- joint larm_module1_dummy_joint: limit effort=0.0 velocity=0.0 -> effort=0.0 velocity=6.5
- joint larm_module2_dummy_joint: limit effort=0.0 velocity=0.0 -> effort=0.0 velocity=6.5
- joint rarm_module1_dummy_joint: limit effort=0.0 velocity=0.0 -> effort=0.0 velocity=6.5
- joint rarm_module2_dummy_joint: limit effort=0.0 velocity=0.0 -> effort=0.0 velocity=6.5
- joint rarm_module2_joint1: limit lower=-1.78 upper=1.78 effort=0.0 velocity=0.0 -> lower=-1.78 upper=1.78 effort=0.0 velocity=6.5

Commit message: Add

File: jedy/jedy_description/urdf/jedy_four_dof.urdf (robot description, URDF)
Before this commit: robot test_robot, 36 links, 35 joints
Links:
- link base_link: geometry collision mesh filename=package://jedy_description/meshes/screw_body_module/base_li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; visual mesh filename=package://jedy_description/meshes/screw_body_module/base_li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
- link head_link0: geometry collision mesh filename=package://jedy_description/meshes/screw_body_module/head_li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; visual mesh filename=package://jedy_description/meshes/screw_body_module/head_li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
- link head_module1_base_link: geometry collision mesh filename=package://jedy_description/meshes/screw_20mmhead_module_cov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; visual mesh filename=package://jedy_description/meshes/screw_20mmhead_module_cov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
- link head_module1_link1: geometry collision mesh filename=package://jedy_description/meshes/screw_20mmhead_module_cov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; visual mesh filename=package://jedy_description/meshes/screw_20mmhead_module_cov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
- link larm_link0: geometry collision mesh filename=package://jedy_description/meshes/screw_body_module/larm_li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; visual mesh filename=package://jedy_description/meshes/screw_body_module/larm_li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
- link larm_module1_base_link: geometry collision mesh filename=package://jedy_description/meshes/screw_crosscantileverleft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; visual mesh filename=package://jedy_description/meshes/screw_crosscantileverleft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
- link larm_module1_link1: geometry collision mesh filename=package://jedy_description/meshes/screw_crosscantileverleft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; visual mesh filename=package://jedy_description/meshes/screw_crosscantileverleft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
- link larm_module1_link2: geometry collision mesh filename=package://jedy_description/meshes/screw_crosscantileverleft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; visual mesh filename=package://jedy_description/meshes/screw_crosscantileverleft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
- link larm_module2_base_link: geometry collision mesh filename=package://jedy_description/meshes/screw_26mmhinge_module_co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; visual mesh filename=package://jedy_description/meshes/screw_26mmhinge_module_co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
- link larm_module2_link1: geometry collision mesh filename=package://jedy_description/meshes/screw_26mmhinge_module_co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; visual mesh filename=package://jedy_description/meshes/screw_26mmhinge_module_co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
- link left_hand_base_link: geometry collision mesh filename=package://jedy_description/meshes/screw_hand_module/base_li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; visual mesh filename=package://jedy_description/meshes/screw_hand_module/base_li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
- link left_hand_link1: geometry collision mesh filename=package://jedy_description/meshes/screw_hand_module/link1.d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; visual mesh filename=package://jedy_description/meshes/screw_hand_module/link1.d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
- link left_hand_link2: geometry collision mesh filename=package://jedy_description/meshes/screw_hand_module/link2.d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; visual mesh filename=package://jedy_description/meshes/screw_hand_module/link2.d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
- link mechanum_base_link: geometry collision cylinder length=0.02 radius=0.03; visual mesh filename=package://jedy_description/meshes/screw_mechanum_module/bas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
- link mechanum_link1: geometry collision cylinder length=0.02 radius=0.03; visual mesh filename=package://jedy_description/meshes/screw_mechanum_module/lin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
- link mechanum_link2: geometry collision cylinder length=0.02 radius=0.03; visual mesh filename=package://jedy_description/meshes/screw_mechanum_module/lin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
- link mechanum_link3: geometry collision cylinder length=0.02 radius=0.03; visual mesh filename=package://jedy_description/meshes/screw_mechanum_module/lin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
- link mechanum_link4: geometry collision cylinder length=0.02 radius=0.03; visual mesh filename=package://jedy_description/meshes/screw_mechanum_module/lin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
- link rarm_link0: geometry collision mesh filename=package://jedy_description/meshes/screw_body_module/rarm_li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; visual mesh filename=package://jedy_description/meshes/screw_body_module/rarm_li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
- link rarm_module1_base_link: geometry collision mesh filename=package://jedy_description/meshes/screw_crosscantileverrigh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; visual mesh filename=package://jedy_description/meshes/screw_crosscantileverrigh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
- link rarm_module1_link1: geometry collision mesh filename=package://jedy_description/meshes/screw_crosscantileverrigh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; visual mesh filename=package://jedy_description/meshes/screw_crosscantileverrigh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
- link rarm_module1_link2: geometry collision mesh filename=package://jedy_description/meshes/screw_crosscantileverrigh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; visual mesh filename=package://jedy_description/meshes/screw_crosscantileverrigh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
- link rarm_module2_base_link: geometry collision mesh filename=package://jedy_description/meshes/screw_26mmhinge_module_co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; visual mesh filename=package://jedy_description/meshes/screw_26mmhinge_module_co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
- link rarm_module2_link1: geometry collision mesh filename=package://jedy_description/meshes/screw_26mmhinge_module_co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; visual mesh filename=package://jedy_description/meshes/screw_26mmhinge_module_co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
- link right_hand_base_link: geometry collision mesh filename=package://jedy_description/meshes/screw_hand_module/base_li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; visual mesh filename=package://jedy_description/meshes/screw_hand_module/base_li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
- link right_hand_link1: geometry collision mesh filename=package://jedy_description/meshes/screw_hand_module/link1.d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; visual mesh filename=package://jedy_description/meshes/screw_hand_module/link1.d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
- link right_hand_link2: geometry collision mesh filename=package://jedy_description/meshes/screw_hand_module/link2.d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; visual mesh filename=package://jedy_description/meshes/screw_hand_module/link2.d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

Commit message: Reduce mesh size

File: jedy/jedy_description/urdf/jedy_four_dof.urdf (robot description, URDF)
Before this commit: robot test_robot, 36 links, 35 joints
Joints:
- joint dummy_joint_larm: origin xyz=0.0 0.0135 0.0 rpy=-1.5707963267949003 -0.0 0.0 -> xyz=0.0 0.0135 0.0 rpy=-1.5707963267949006 -0.0 0.0
- joint dummy_joint_rarm: origin xyz=0.0 -0.0135 0.0 rpy=1.5707963267949003 -0.0 0.0 -> xyz=0.0 -0.0135 0.0 rpy=1.5707963267949006 -0.0 0.0
- joint head_module1_base_link_to_dummy_link_head_joint: axis (none) -> 1. 0. 0.; limit (none) -> effort=0.0 velocity=0.0; origin xyz=0 0 0 rpy=0 0 0 -> xyz=0.0 0.0 0.0 rpy=0.0 -0.0 0.0
- joint larm_module1_base_link_to_dummy_link_larm_joint: axis (none) -> 1. 0. 0.; limit (none) -> effort=0.0 velocity=0.0; origin xyz=0 0 0 rpy=0 0 -1.5707963267948966 -> xyz=0.0 0.0 0.0 rpy=-0.0 -0.0 -1.5707963267948963
- joint larm_module1_dummy_joint: origin xyz=-0.031 0.0 0.0 rpy=-3.353553828779909e-15 1.5707963267948932 3.141592653589793 -> xyz=-0.031 0.0 0.0 rpy=-3.3535538287799086e-15 1.5707963267948932 3.141592653589793
- joint larm_module2_base_link_to_larm_module1_dummy_link_joint: axis (none) -> 1. 0. 0.; limit (none) -> effort=0.0 velocity=0.0; origin xyz=0 0 0 rpy=0 0 0 -> xyz=0.0 0.0 0.0 rpy=0.0 -0.0 0.0
- joint left_hand_base_link_to_larm_module2_dummy_link_joint: axis (none) -> 1. 0. 0.; limit (none) -> effort=0.0 velocity=0.0; origin xyz=0 0 0 rpy=0 0 0 -> xyz=0.0 0.0 0.0 rpy=0.0 -0.0 0.0
- joint mechanum_base_link_to_dummy_link_rleg_joint: axis (none) -> 1. 0. 0.; limit (none) -> effort=0.0 velocity=0.0; origin xyz=0 0 0 rpy=0 0 0 -> xyz=0.0 0.0 0.0 rpy=0.0 -0.0 0.0
- joint rarm_module1_base_link_to_dummy_link_rarm_joint: axis (none) -> 1. 0. 0.; limit (none) -> effort=0.0 velocity=0.0; origin xyz=0 0 0 rpy=0 0 -1.5707963267948966 -> xyz=0.0 0.0 0.0 rpy=-0.0 -0.0 -1.5707963267948963
- joint rarm_module2_base_link_to_rarm_module1_dummy_link_joint: axis (none) -> 1. 0. 0.; limit (none) -> effort=0.0 velocity=0.0; origin xyz=0 0 0 rpy=0 0 0 -> xyz=0.0 0.0 0.0 rpy=0.0 -0.0 0.0
- joint right_hand_base_link_to_rarm_module2_dummy_link_joint: axis (none) -> 1. 0. 0.; limit (none) -> effort=0.0 velocity=0.0; origin xyz=0 0 0 rpy=0 0 0 -> xyz=0.0 0.0 0.0 rpy=0.0 -0.0 0.0

Commit message: Add

File: jedy/jedy_description/urdf/jedy_four_dof.urdf (robot description, URDF)
Before this commit: robot test_robot, 36 links, 35 joints
Links:
- link base_link: geometry collision mesh filename=model://jedy_description/meshes/screw_body_module/base_link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; visual mesh filename=model://jedy_description/meshes/screw_body_module/base_link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
- link head_link0: geometry collision mesh filename=model://jedy_description/meshes/screw_body_module/head_link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; visual mesh filename=model://jedy_description/meshes/screw_body_module/head_link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
- link head_module1_base_link: geometry collision mesh filename=model://jedy_description/meshes/screw_20mmhead_module_cover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; visual mesh filename=model://jedy_description/meshes/screw_20mmhead_module_cover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
- link head_module1_link1: geometry collision mesh filename=model://jedy_description/meshes/screw_20mmhead_module_cover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; visual mesh filename=model://jedy_description/meshes/screw_20mmhead_module_cover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
- link larm_link0: geometry collision mesh filename=model://jedy_description/meshes/screw_body_module/larm_link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; visual mesh filename=model://jedy_description/meshes/screw_body_module/larm_link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
- link larm_module1_base_link: geometry collision mesh filename=model://jedy_description/meshes/screw_crosscantileverleft_m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; visual mesh filename=model://jedy_description/meshes/screw_crosscantileverleft_m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
- link larm_module1_link1: geometry collision mesh filename=model://jedy_description/meshes/screw_crosscantileverleft_m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; visual mesh filename=model://jedy_description/meshes/screw_crosscantileverleft_m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
- link larm_module1_link2: geometry collision mesh filename=model://jedy_description/meshes/screw_crosscantileverleft_m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; visual mesh filename=model://jedy_description/meshes/screw_crosscantileverleft_m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
- link larm_module2_base_link: geometry collision mesh filename=model://jedy_description/meshes/screw_26mmhinge_module_cove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; visual mesh filename=model://jedy_description/meshes/screw_26mmhinge_module_cove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
- link larm_module2_link1: geometry collision mesh filename=model://jedy_description/meshes/screw_26mmhinge_module_cove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; visual mesh filename=model://jedy_description/meshes/screw_26mmhinge_module_cove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
- link left_hand_base_link: geometry collision mesh filename=model://jedy_description/meshes/screw_hand_module/base_link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; visual mesh filename=model://jedy_description/meshes/screw_hand_module/base_link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
- link left_hand_link1: geometry collision mesh filename=model://jedy_description/meshes/screw_hand_module/link1.dae; visual mesh filename=model://jedy_description/meshes/screw_hand_module/link1.dae
- link left_hand_link2: geometry collision mesh filename=model://jedy_description/meshes/screw_hand_module/link2.dae; visual mesh filename=model://jedy_description/meshes/screw_hand_module/link2.dae
- link mechanum_base_link: geometry collision cylinder length=0.02 radius=0.03; visual mesh filename=model://jedy_description/meshes/screw_mechanum_module/base_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
- link mechanum_link1: geometry collision cylinder length=0.02 radius=0.03; visual mesh filename=model://jedy_description/meshes/screw_mechanum_module/link1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
- link mechanum_link2: geometry collision cylinder length=0.02 radius=0.03; visual mesh filename=model://jedy_description/meshes/screw_mechanum_module/link2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
- link mechanum_link3: geometry collision cylinder length=0.02 radius=0.03; visual mesh filename=model://jedy_description/meshes/screw_mechanum_module/link3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
- link mechanum_link4: geometry collision cylinder length=0.02 radius=0.03; visual mesh filename=model://jedy_description/meshes/screw_mechanum_module/link4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
- link rarm_link0: geometry collision mesh filename=model://jedy_description/meshes/screw_body_module/rarm_link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; visual mesh filename=model://jedy_description/meshes/screw_body_module/rarm_link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
- link rarm_module1_base_link: geometry collision mesh filename=model://jedy_description/meshes/screw_crosscantileverright_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; visual mesh filename=model://jedy_description/meshes/screw_crosscantileverright_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
- link rarm_module1_link1: geometry collision mesh filename=model://jedy_description/meshes/screw_crosscantileverright_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; visual mesh filename=model://jedy_description/meshes/screw_crosscantileverright_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
- link rarm_module1_link2: geometry collision mesh filename=model://jedy_description/meshes/screw_crosscantileverright_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; visual mesh filename=model://jedy_description/meshes/screw_crosscantileverright_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
- link rarm_module2_base_link: geometry collision mesh filename=model://jedy_description/meshes/screw_26mmhinge_module_cove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; visual mesh filename=model://jedy_description/meshes/screw_26mmhinge_module_cove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
- link rarm_module2_link1: geometry collision mesh filename=model://jedy_description/meshes/screw_26mmhinge_module_cove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; visual mesh filename=model://jedy_description/meshes/screw_26mmhinge_module_cove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
- link right_hand_base_link: geometry collision mesh filename=model://jedy_description/meshes/screw_hand_module/base_link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; visual mesh filename=model://jedy_description/meshes/screw_hand_module/base_link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
- link right_hand_link1: geometry collision mesh filename=model://jedy_description/meshes/screw_hand_module/link1.dae; visual mesh filename=model://jedy_description/meshes/screw_hand_module/link1.dae
- link right_hand_link2: geometry collision mesh filename=model://jedy_description/meshes/screw_hand_module/link2.dae; visual mesh filename=model://jedy_description/meshes/screw_hand_module/link2.dae

Commit message: Add

File: jedy/jedy_description/urdf/jedy_four_dof.urdf (robot description, URDF)
Before this commit: robot test_robot, 36 links, 35 joints
Links:
- link base_link: geometry collision mesh filename=package://jedy_description/meshes/screw_body_module/base_li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; visual mesh filename=package://jedy_description/meshes/screw_body_module/base_li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
- link head_link0: mass 0.0139002702415607 -> 0.1; geometry collision mesh filename=package://jedy_description/meshes/screw_body_module/head_li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; visual mesh filename=package://jedy_description/meshes/screw_body_module/head_li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
- link head_module1_base_link: geometry collision mesh filename=package://jedy_description/meshes/screw_20mmhead_module_cov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; visual mesh filename=package://jedy_description/meshes/screw_20mmhead_module_cov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
- link head_module1_link1: geometry collision mesh filename=package://jedy_description/meshes/screw_20mmhead_module_cov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; visual mesh filename=package://jedy_description/meshes/screw_20mmhead_module_cov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
- link larm_link0: mass 0.0139002702415604 -> 0.1; geometry collision mesh filename=package://jedy_description/meshes/screw_body_module/larm_li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; visual mesh filename=package://jedy_description/meshes/screw_body_module/larm_li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
- link larm_module1_base_link: mass 0.0119463231340018 -> 0.05; geometry collision mesh filename=package://jedy_description/meshes/screw_crosscantileverleft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; visual mesh filename=package://jedy_description/meshes/screw_crosscantileverleft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
- link larm_module1_link1: geometry collision mesh filename=package://jedy_description/meshes/screw_crosscantileverleft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; visual mesh filename=package://jedy_description/meshes/screw_crosscantileverleft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
- link larm_module1_link2: geometry collision mesh filename=package://jedy_description/meshes/screw_crosscantileverleft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; visual mesh filename=package://jedy_description/meshes/screw_crosscantileverleft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
- link larm_module2_base_link: mass 0.038356588287215 -> 0.15; geometry collision mesh filename=package://jedy_description/meshes/screw_26mmhinge_module_co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; visual mesh filename=package://jedy_description/meshes/screw_26mmhinge_module_co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
- link larm_module2_link1: mass 0.0156652005671847 -> 0.08; geometry collision mesh filename=package://jedy_description/meshes/screw_26mmhinge_module_co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; visual mesh filename=package://jedy_description/meshes/screw_26mmhinge_module_co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
- link left_hand_base_link: mass 0.0323742495584158 -> 0.12; geometry collision mesh filename=package://jedy_description/meshes/screw_hand_module/base_li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; visual mesh filename=package://jedy_description/meshes/screw_hand_module/base_li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
- link left_hand_link1: mass 0.00827607897427458 -> 0.05; geometry collision mesh filename=package://jedy_description/meshes/screw_hand_module/link1.d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; visual mesh filename=package://jedy_description/meshes/screw_hand_module/link1.d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
- link left_hand_link2: mass 0.00827607897427456 -> 0.05; geometry collision mesh filename=package://jedy_description/meshes/screw_hand_module/link2.d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; visual mesh filename=package://jedy_description/meshes/screw_hand_module/link2.d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
- link mechanum_base_link: geometry collision cylinder length=0.02 radius=0.03; visual mesh filename=package://jedy_description/meshes/screw_mechanum_module/bas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
- link mechanum_link1: geometry collision cylinder length=0.02 radius=0.03; visual mesh filename=package://jedy_description/meshes/screw_mechanum_module/lin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
- link mechanum_link2: geometry collision cylinder length=0.02 radius=0.03; visual mesh filename=package://jedy_description/meshes/screw_mechanum_module/lin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
- link mechanum_link3: geometry collision cylinder length=0.02 radius=0.03; visual mesh filename=package://jedy_description/meshes/screw_mechanum_module/lin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
- link mechanum_link4: geometry collision cylinder length=0.02 radius=0.03; visual mesh filename=package://jedy_description/meshes/screw_mechanum_module/lin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
- link rarm_link0: mass 0.0139002702415581 -> 0.1; geometry collision mesh filename=package://jedy_description/meshes/screw_body_module/rarm_li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; visual mesh filename=package://jedy_description/meshes/screw_body_module/rarm_li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
- link rarm_module1_base_link: mass 0.0119463231340018 -> 0.05; geometry collision mesh filename=package://jedy_description/meshes/screw_crosscantileverrigh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; visual mesh filename=package://jedy_description/meshes/screw_crosscantileverrigh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
- link rarm_module1_link1: mass 0.0552019977106494 -> 0.2; geometry collision mesh filename=package://jedy_description/meshes/screw_crosscantileverrigh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; visual mesh filename=package://jedy_description/meshes/screw_crosscantileverrigh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
- link rarm_module1_link2: mass 0.0139002702415665 -> 0.1; geometry collision mesh filename=package://jedy_description/meshes/screw_crosscantileverrigh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; visual mesh filename=package://jedy_description/meshes/screw_crosscantileverrigh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
- link rarm_module2_base_link: mass 0.038356588287215 -> 0.15; geometry collision mesh filename=package://jedy_description/meshes/screw_26mmhinge_module_co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; visual mesh filename=package://jedy_description/meshes/screw_26mmhinge_module_co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
- link rarm_module2_link1: mass 0.0156652005671847 -> 0.08; geometry collision mesh filename=package://jedy_description/meshes/screw_26mmhinge_module_co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; visual mesh filename=package://jedy_description/meshes/screw_26mmhinge_module_co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
- link right_hand_base_link: mass 0.0323742495584158 -> 0.12; geometry collision mesh filename=package://jedy_description/meshes/screw_hand_module/base_li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; visual mesh filename=package://jedy_description/meshes/screw_hand_module/base_li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
- link right_hand_link1: mass 0.00827607897427458 -> 0.05; geometry collision mesh filename=package://jedy_description/meshes/screw_hand_module/link1.d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; visual mesh filename=package://jedy_description/meshes/screw_hand_module/link1.d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
- link right_hand_link2: mass 0.00827607897427456 -> 0.05; geometry collision mesh filename=package://jedy_description/meshes/screw_hand_module/link2.d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; visual mesh filename=package://jedy_description/meshes/screw_hand_module/link2.d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

Commit message: Add

File: jedy/jedy_description/urdf/jedy_four_dof.urdf (robot description, URDF)
Before this commit: robot test_robot, 36 links, 35 joints
Links:
- link mechanum_link1: geometry collision mesh filename=package://jedy_description/meshes/screw_mechanum_module/lin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; visual mesh filename=package://jedy_description/meshes/screw_mechanum_module/lin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
- link mechanum_link2: geometry collision mesh filename=package://jedy_description/meshes/screw_mechanum_module/lin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; visual mesh filename=package://jedy_description/meshes/screw_mechanum_module/lin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
- link mechanum_link3: geometry collision mesh filename=package://jedy_description/meshes/screw_mechanum_module/lin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; visual mesh filename=package://jedy_description/meshes/screw_mechanum_module/lin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
- link mechanum_link4: geometry collision mesh filename=package://jedy_description/meshes/screw_mechanum_module/lin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; visual mesh filename=package://jedy_description/meshes/screw_mechanum_module/lin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
