Commit message: Add

File: jedy/jedy_description/urdf/jedy_four_dof.urdf (robot description, URDF)
Before this commit: robot test_robot, 36 links, 35 joints
Links:
- link mechanum_base_link: geometry collision mesh filename=package://jedy_description/meshes/screw_mechanum_module/bas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; visual mesh filename=package://jedy_description/meshes/screw_mechanum_module/bas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

Commit message: Add

File: jedy/jedy_description/urdf/jedy_four_dof.urdf (robot description, URDF)
Before this commit: robot test_robot, 36 links, 35 joints
Links:
- link mechanum_link1: geometry collision cylinder length=0.03370000049471855 radius=0.025114329531788826; visual mesh filename=package://jedy_description/meshes/screw_mechanum_module/lin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
- link mechanum_link2: geometry collision cylinder length=0.03370000049471855 radius=0.025114329531788826; visual mesh filename=package://jedy_description/meshes/screw_mechanum_module/lin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
- link mechanum_link3: geometry collision cylinder length=0.03370000049471855 radius=0.025114329531788826; visual mesh filename=package://jedy_description/meshes/screw_mechanum_module/lin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
- link mechanum_link4: geometry collision cylinder length=0.03370000049471855 radius=0.025114329531788826; visual mesh filename=package://jedy_description/meshes/screw_mechanum_module/lin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
