Commit message: Fixing link name and remove real_base_link

File: jedy/jedy_description/urdf/jedy.urdf (robot description, URDF)
Before this commit: robot jedy, 32 links, 31 joints
Links:
- removed link real_base_link
- link base_link: mass None -> 0.671312; geometry collision mesh filename=package://jedy_description/meshes/base_link.stl; visual mesh filename=package://jedy_description/meshes/base_link.dae
Joints:
- removed joint pseudo_base_joint
- joint front_left_wheel_joint: parent real_base_link -> base_link
- joint front_right_wheel_joint: parent real_base_link -> base_link
- joint head_joint0: parent real_base_link -> base_link
- joint larm_joint0: parent real_base_link -> base_link
- joint rarm_joint0: parent real_base_link -> base_link
- joint rear_left_wheel_joint: parent real_base_link -> base_link
- joint rear_right_wheel_joint: parent real_base_link -> base_link
