Commit message: Add

File: jedy/jedy_description/urdf/jedy_gz.xacro (robot description, xacro)
@@ -690,5 +690,5 @@
     <child link="camera_link"/>
     <axis xyz="1. 0. 0."/>
-    <origin xyz="0.0 0.005 0.05" rpy="0.0 -0.0 0.0"/>
+    <origin xyz="0.0 0.015 0.08" rpy="0.0 -0.0 0.0"/>
   </joint>
   <joint name="camera_color_frame_joint" type="fixed">

Commit message: Add

File: jedy/jedy_description/urdf/jedy_gz.xacro (robot description, xacro)
@@ -16,7 +16,7 @@
     <collision>
       <geometry>
-        <mesh filename="package://jedy_description/meshes/base_link.stl"/>
-      </geometry>
-      <origin xyz="0.0 0.0 0.0" rpy="0.0 -0.0 0.0"/>
+        <box size="0.200 0.200 0.100"/>
+      </geometry>
+      <origin xyz="0.0 0.0 0.021" rpy="0.0 0.0 0.0"/>
     </collision>
   </link>
@@ -36,7 +36,7 @@
     <collision>
       <geometry>
-        <mesh filename="package://jedy_description/meshes/rarm_link0.stl"/>
-      </geometry>
-      <origin xyz="0.0 0.0 0.0" rpy="0.0 -0.0 0.0"/>
+        <cylinder radius="0.015" length="0.035"/>
+      </geometry>
+      <origin xyz="0.0075 0.05 -0.077" rpy="0.0 0.0 0.0"/>
     </collision>
   </link>
@@ -55,7 +55,7 @@
     <collision>
       <geometry>
-        <mesh filename="package://jedy_description/meshes/rarm_link1.stl"/>
-      </geometry>
-      <origin xyz="0.0 0.0 0.0" rpy="0.0 -0.0 0.0"/>
+        <cylinder radius="0.018" length="0.025"/>
+      </geometry>
+      <origin xyz="0.006 0.063 -0.076" rpy="0.0 0.0 0.0"/>
     </collision>
   </link>
@@ -74,7 +74,7 @@
     <collision>
       <geometry>
-        <mesh filename="package://jedy_description/meshes/rarm_link2.stl"/>
-      </geometry>
-      <origin xyz="0.0 0.0 0.0" rpy="0.0 -0.0 0.0"/>
+        <cylinder radius="0.018" length="0.040"/>
+      </geometry>
+      <origin xyz="-0.014 0.079 -0.051" rpy="0.0 0.0 0.0"/>
     </collision>
   </link>
@@ -93,7 +93,7 @@
     <collision>
       <geometry>
-        <mesh filename="package://jedy_description/meshes/rarm_link3.stl"/>
-      </geometry>
-      <origin xyz="0.0 0.0 0.0" rpy="0.0 -0.0 0.0"/>
+        <cylinder radius="0.020" length="0.080"/>
+      </geometry>
+      <origin xyz="-0.042 0.079 -0.023" rpy="0.0 0.0 0.0"/>
     </collision>
   </link>
@@ -112,7 +112,7 @@
     <collision>
       <geometry>
-        <mesh filename="package://jedy_description/meshes/rarm_link4.stl"/>
-      </geometry>
-      <origin xyz="0.0 0.0 0.0" rpy="0.0 -0.0 0.0"/>
+        <cylinder radius="0.015" length="0.030"/>
+      </geometry>
+      <origin xyz="0.002 0.078 0.057" rpy="0.0 0.0 0.0"/>
     </collision>
   </link>
@@ -131,7 +131,7 @@
     <collision>
       <geometry>
-        <mesh filename="package://jedy_description/meshes/rarm_link5.stl"/>
-      </geometry>
-      <origin xyz="0.0 0.0 0.0" rpy="0.0 -0.0 0.0"/>
+        <cylinder radius="0.018" length="0.028"/>
+      </geometry>
+      <origin xyz="-0.0005 0.062 0.082" rpy="0.0 0.0 0.0"/>
     </collision>
   </link>
@@ -150,7 +150,7 @@
     <collision>
       <geometry>
-        <mesh filename="package://jedy_description/meshes/rarm_link6.stl"/>
-      </geometry>
-      <origin xyz="0.0 0.0 0.0" rpy="0.0 -0.0 0.0"/>
+        <cylinder radius="0.020" length="0.025"/>
+      </geometry>
+      <origin xyz="-0.033 0.077 0.101" rpy="0.0 0.0 0.0"/>
     </collision>
   </link>
@@ -169,7 +169,7 @@
     <collision>
       <geometry>
-        <mesh filename="package://jedy_description/meshes/rarm_link7.stl"/>
-      </geometry>
-      <origin xyz="0.0 0.0 0.0" rpy="0.0 -0.0 0.0"/>
+        <box size="0.012 0.030 0.060"/>
+      </geometry>
+      <origin xyz="-0.006 0.091 0.155" rpy="0.0 0.0 0.0"/>
     </collision>
   </link>
@@ -188,7 +188,7 @@
     <collision>
       <geometry>
-        <mesh filename="package://jedy_description/meshes/rarm_link8.stl"/>
-      </geometry>
-      <origin xyz="0.0 0.0 0.0" rpy="0.0 -0.0 0.0"/>
+        <box size="0.012 0.030 0.060"/>
+      </geometry>
+      <origin xyz="-0.006 0.065 0.166" rpy="0.0 0.0 0.0"/>
     </collision>
   </link>
@@ -207,7 +207,7 @@
     <collision>
       <geometry>
-        <mesh filename="package://jedy_description/meshes/larm_link0.stl"/>
-      </geometry>
-      <origin xyz="0.0 0.0 0.0" rpy="0.0 -0.0 0.0"/>
+        <cylinder radius="0.015" length="0.035"/>
+      </geometry>
+      <origin xyz="0.0075 0.05 0.077" rpy="0.0 0.0 0.0"/>
     </collision>
   </link>
@@ -226,7 +226,7 @@
     <collision>
       <geometry>
-        <mesh filename="package://jedy_description/meshes/larm_link1.stl"/>
-      </geometry>
-      <origin xyz="0.0 0.0 0.0" rpy="0.0 -0.0 0.0"/>
+        <cylinder radius="0.018" length="0.025"/>
+      </geometry>
+      <origin xyz="0.007 -0.094 -0.061" rpy="0.0 0.0 0.0"/>
     </collision>
   </link>
@@ -245,7 +245,7 @@
     <collision>
       <geometry>
-        <mesh filename="package://jedy_description/meshes/larm_link2.stl"/>
-      </geometry>
-      <origin xyz="0.0 0.0 0.0" rpy="0.0 -0.0 0.0"/>
+        <cylinder radius="0.018" length="0.040"/>
+      </geometry>
+      <origin xyz="-0.014 -0.079 -0.051" rpy="0.0 0.0 0.0"/>
     </collision>
   </link>
@@ -264,7 +264,7 @@
     <collision>
       <geometry>
-        <mesh filename="package://jedy_description/meshes/larm_link3.stl"/>
-      </geometry>
-      <origin xyz="0.0 0.0 0.0" rpy="0.0 -0.0 0.0"/>
+        <cylinder radius="0.020" length="0.080"/>
+      </geometry>
+      <origin xyz="-0.042 -0.079 -0.013" rpy="0.0 0.0 0.0"/>
     </collision>
   </link>
@@ -283,7 +283,7 @@
     <collision>
       <geometry>
-        <mesh filename="package://jedy_description/meshes/larm_link4.stl"/>
-      </geometry>
-      <origin xyz="0.0 0.0 0.0" rpy="0.0 -0.0 0.0"/>
+        <cylinder radius="0.015" length="0.030"/>
+      </geometry>
+      <origin xyz="0.002 -0.078 0.057" rpy="0.0 0.0 0.0"/>
     </collision>
   </link>
@@ -302,7 +302,7 @@
     <collision>
       <geometry>
-        <mesh filename="package://jedy_description/meshes/larm_link5.stl"/>
-      </geometry>
-      <origin xyz="0.0 0.0 0.0" rpy="0.0 -0.0 0.0"/>
+        <cylinder radius="0.018" length="0.028"/>
+      </geometry>
+      <origin xyz="-0.0005 -0.093 0.083" rpy="0.0 0.0 0.0"/>
     </collision>
   </link>
@@ -321,7 +321,7 @@
     <collision>
       <geometry>
-        <mesh filename="package://jedy_description/meshes/larm_link6.stl"/>
-      </geometry>
-      <origin xyz="0.0 0.0 0.0" rpy="0.0 -0.0 0.0"/>
+        <cylinder radius="0.020" length="0.025"/>
+      </geometry>
+      <origin xyz="-0.033 -0.078 0.107" rpy="0.0 0.0 0.0"/>
     </collision>
   </link>
@@ -340,7 +340,7 @@
     <collision>
       <geometry>
-        <mesh filename="package://jedy_description/meshes/larm_link7.stl"/>
-      </geometry>
-      <origin xyz="0.0 0.0 0.0" rpy="0.0 -0.0 0.0"/>
+        <box size="0.012 0.030 0.060"/>
+      </geometry>
+      <origin xyz="-0.006 -0.091 0.166" rpy="0.0 0.0 0.0"/>
     </collision>
   </link>
@@ -359,7 +359,7 @@
     <collision>
       <geometry>
-        <mesh filename="package://jedy_description/meshes/larm_link8.stl"/>
-      </geometry>
-      <origin xyz="0.0 0.0 0.0" rpy="0.0 -0.0 0.0"/>
+        <box size="0.012 0.030 0.060"/>
+      </geometry>
+      <origin xyz="-0.006 -0.065 0.155" rpy="0.0 0.0 0.0"/>
     </collision>
   </link>
@@ -378,7 +378,7 @@
     <collision>
       <geometry>
-        <mesh filename="package://jedy_description/meshes/head_link0.stl"/>
-      </geometry>
-      <origin xyz="0.0 0.0 0.0" rpy="0.0 -0.0 0.0"/>
+        <cylinder radius="0.025" length="0.040"/>
+      </geometry>
+      <origin xyz="0.0 0.0 0.023" rpy="0.0 0.0 0.0"/>
     </collision>
   </link>
@@ -397,7 +397,7 @@
     <collision>
       <geometry>
-        <mesh filename="package://jedy_description/meshes/head_link1.stl"/>
-      </geometry>
-      <origin xyz="0.0 0.0 0.0" rpy="0.0 -0.0 0.0"/>
+        <box size="0.070 0.070 0.150"/>
+      </geometry>
+      <origin xyz="-0.001 0.0 0.186" rpy="0.0 0.0 0.0"/>
     </collision>
   </link>
@@ -750,5 +750,5 @@
       <pose>0 0 0 0 0 0</pose>
       <visualize>true</visualize>
-      <update_rate>10</update_rate>
+      <update_rate>8</update_rate>
       <topic>/scan_raw</topic>
       <gz:frame_id xmlns:gz="http://sdformat.org/schemas/sensor">base_laser</gz:frame_id>
@@ -764,5 +764,5 @@
         <range>
           <min>0.12</min>
-          <max>10.0</max>
+          <max>8.0</max>
           <resolution>0.01</resolution>
         </range>
@@ -899,5 +899,5 @@
     <mu1>100.0</mu1>
     <mu2>100.0</mu2>
-    <kp>10000000</kp>
+    <kp>100000</kp>
     <kd>1</kd>
     <maxVel value="100.0"/>
@@ -907,5 +907,5 @@
     <mu1>100.0</mu1>
     <mu2>100.0</mu2>
-    <kp>10000000</kp>
+    <kp>100000</kp>
     <kd>1</kd>
     <maxVel value="100.0"/>
@@ -915,5 +915,5 @@
     <mu1>100.0</mu1>
     <mu2>100.0</mu2>
-    <kp>10000000</kp>
+    <kp>100000</kp>
     <kd>1</kd>
     <maxVel value="100.0"/>
@@ -923,5 +923,5 @@
     <mu1>100.0</mu1>
     <mu2>100.0</mu2>
-    <kp>10000000</kp>
+    <kp>100000</kp>
     <kd>1</kd>
     <maxVel value="100.0"/>
@@ -931,5 +931,5 @@
     <mu1>100.0</mu1>
     <mu2>100.0</mu2>
-    <kp>10000000</kp>
+    <kp>100000</kp>
     <kd>1</kd>
     <material>Gazebo/Yellow</material>
@@ -938,5 +938,5 @@
     <mu1>100.0</mu1>
     <mu2>100.0</mu2>
-    <kp>10000000</kp>
+    <kp>100000</kp>
     <kd>1</kd>
     <material>Gazebo/Yellow</material>
@@ -945,5 +945,5 @@
     <mu1>100.0</mu1>
     <mu2>100.0</mu2>
-    <kp>10000000</kp>
+    <kp>100000</kp>
     <kd>1</kd>
     <material>Gazebo/Yellow</material>
@@ -952,5 +952,5 @@
     <mu1>100.0</mu1>
     <mu2>100.0</mu2>
-    <kp>10000000</kp>
+    <kp>100000</kp>
     <kd>1</kd>
     <material>Gazebo/Yellow</material>
@@ -959,18 +959,18 @@
     <sensor name="camera" type="rgbd_camera">
       <always_on>1</always_on>
-      <update_rate>30</update_rate>
+      <update_rate>15</update_rate>
       <visualize>true</visualize>
       <topic>camera</topic>
       <gz_frame_id>camera_color_optical_frame</gz_frame_id>
       <camera name="camera">
-        <horizontal_fov>1.0471975511965976</horizontal_fov>
+        <horizontal_fov>0.872665</horizontal_fov>
         <image>
-          <width>640</width>
-          <height>480</height>
+          <width>480</width>
+          <height>360</height>
           <format>R8G8B8</format>
         </image>
         <clip>
           <near>0.05</near>
-          <far>10.0</far>
+          <far>8.0</far>
         </clip>
         <noise>
@@ -986,5 +986,5 @@
       <pose>0 0 0 0 0 0</pose>
       <always_on>true</always_on>
-      <update_rate>100</update_rate>
+      <update_rate>50</update_rate>
       <visualize>false</visualize>
       <topic>/imu</topic>
