Commit message: Add

File: jedy/jedy_bringup/urdf/jedy_gazebo_compatible.urdf (robot description, URDF)
Before this commit: robot jedy_robot, 8 links, 7 joints
Joints:
- joint mechanum_joint1: origin xyz=0.08 0.08 -0.05 rpy=0 0 0 -> xyz=0.08 0.08 -0.10 rpy=0 0 0
- joint mechanum_joint2: origin xyz=0.08 -0.08 -0.05 rpy=0 0 0 -> xyz=0.08 -0.08 -0.10 rpy=0 0 0
- joint mechanum_joint3: origin xyz=-0.08 0.08 -0.05 rpy=0 0 0 -> xyz=-0.08 0.08 -0.10 rpy=0 0 0
- joint mechanum_joint4: origin xyz=-0.08 -0.08 -0.05 rpy=0 0 0 -> xyz=-0.08 -0.08 -0.10 rpy=0 0 0
