Commit message: Add

File: jedy/jedy_bringup/urdf/jedy_gz.xacro (robot description, xacro)
@@ -1017,7 +1017,13 @@
     <visual>
       <origin rpy="0 0 1.5707963267948966" xyz="0 0 0"/>
+      <geometry>
+        <box size="0.015 0.13 0.022"/>
+      </geometry>
     </visual>
     <collision>
       <origin rpy="0 0 0" xyz="0.0 0.0 0.0"/>
+      <geometry>
+        <box size="0.015 0.13 0.022"/>
+      </geometry>
     </collision>
     <inertial>
@@ -1035,41 +1041,31 @@
   <link name="camera_depth_optical_frame"></link>
   <joint name="camera_depth_optical_frame_joint" type="fixed"> <origin rpy="-1.57 0 -1.57" xyz="0 0 0"/> <parent link="camera_depth_frame"/> <child link="camera_depth_optical_frame"/> </joint>
-  <!-- Camera sensor commented out - Gazebo Classic plugin not compatible with Gazebo Harmonic -->
-  <!-- <gazebo reference="camera_link"> -->
-  <!--   <sensor name="camera" type="depth"> -->
-  <!--     <always_on>true</always_on> -->
-  <!--     <update_rate>5.0</update_rate> -->
-  <!--     <camera> -->
-  <!--       <horizontal_fov>1.0471975511965976</horizontal_fov> -->
-  <!--       <image> -->
-  <!--         <format>B8G8R8</format> -->
-  <!--         <width>640</width> -->
-  <!--         <height>480</height> -->
-  <!--       </image> -->
-  <!--       <clip> -->
-  <!--         <near>0.05</near> -->
-  <!--         <far>8.0</far> -->
-  <!--       </clip> -->
-  <!--     </camera> -->
-  <!--     <plugin filename="libgazebo_ros_openni_kinect.so" name="kinect_camera_controller"> -->
-  <!--       <cameraName>camera</cameraName> -->
-  <!--       <alwaysOn>true</alwaysOn> -->
-  <!--       <updateRate>5</updateRate> -->
-  <!--       <imageTopicName>rgb/image_raw</imageTopicName> -->
-  <!--       <depthImageTopicName>depth/image_raw</depthImageTopicName> -->
-  <!--       <pointCloudTopicName>depth/points</pointCloudTopicName> -->
-  <!--       <cameraInfoTopicName>rgb/camera_info</cameraInfoTopicName> -->
-  <!--       <depthImageCameraInfoTopicName>depth/camera_info</depthImageCameraInfoTopicName> -->
-  <!--       <frameName>camera_depth_optical_frame</frameName> -->
-  <!--       <baseline>0.1</baseline> -->
-  <!--       <distortion_k1>0.0</distortion_k1> -->
-  <!--       <distortion_k2>0.0</distortion_k2> -->
-  <!--       <distortion_k3>0.0</distortion_k3> -->
-  <!--       <distortion_t1>0.0</distortion_t1> -->
-  <!--       <distortion_t2>0.0</distortion_t2> -->
-  <!--       <pointCloudCutoff>0.4</pointCloudCutoff> -->
-  <!--     </plugin> -->
-  <!--   </sensor> -->
-  <!-- </gazebo> -->
+  <!-- RGBD Camera sensor for Gazebo Harmonic (outputs RGB, depth, and point cloud) -->
+  <gazebo reference="camera_link">
+    <sensor name="camera" type="rgbd_camera">
+      <always_on>1</always_on>
+      <update_rate>30</update_rate>
+      <visualize>true</visualize>
+      <topic>camera</topic>
+      <frame_id>camera_depth_optical_frame</frame_id>
+      <camera name="camera">
+        <horizontal_fov>1.0471975511965976</horizontal_fov>
+        <image>
+          <width>640</width>
+          <height>480</height>
+          <format>R8G8B8</format>
+        </image>
+        <clip>
+          <near>0.05</near>
+          <far>10.0</far>
+        </clip>
+        <noise>
+          <type>gaussian</type>
+          <mean>0.0</mean>
+          <stddev>0.007</stddev>
+        </noise>
+      </camera>
+    </sensor>
+  </gazebo>
   <ros2_control name="GazeboSimSystem" type="system">
     <hardware>
