Commit message: Add

File: jedy/jedy_bringup/urdf/jedy_gz_diffdrive.xacro (robot description, xacro)
@@ -1095,5 +1095,36 @@
       <plugin>gz_ros2_control/GazeboSimSystem</plugin>
     </hardware>
-    <!-- Wheel joints removed - now controlled by DiffDrive plugin -->
+    <joint name="front_left_wheel_joint">
+      <command_interface name="velocity">
+        <param name="min">-10</param>
+        <param name="max">10</param>
+      </command_interface>
+      <state_interface name="velocity"/>
+      <state_interface name="position"/>
+    </joint>
+    <joint name="front_right_wheel_joint">
+      <command_interface name="velocity">
+        <param name="min">-10</param>
+        <param name="max">10</param>
+      </command_interface>
+      <state_interface name="velocity"/>
+      <state_interface name="position"/>
+    </joint>
+    <joint name="rear_left_wheel_joint">
+      <command_interface name="velocity">
+        <param name="min">-10</param>
+        <param name="max">10</param>
+      </command_interface>
+      <state_interface name="velocity"/>
+      <state_interface name="position"/>
+    </joint>
+    <joint name="rear_right_wheel_joint">
+      <command_interface name="velocity">
+        <param name="min">-10</param>
+        <param name="max">10</param>
+      </command_interface>
+      <state_interface name="velocity"/>
+      <state_interface name="position"/>
+    </joint>
     <joint name="head_joint0">
       <command_interface name="position">
@@ -1279,23 +1310,7 @@
   <!-- Gazebo plugins -->
   <gazebo>
-    <!-- ros2_control plugin for arm and head joints -->
     <plugin filename="gz_ros2_control-system" name="gz_ros2_control::GazeboSimROS2ControlPlugin">
       <parameters>/home/iory/ros2/enshu/install/jedy_bringup/share/jedy_bringup/config/jedy_controllers.ros2.yaml</parameters>
     </plugin>
-    <!-- DiffDrive plugin for base mobility (using rear wheels) -->
-    <plugin filename="gz-sim-diff-drive-system" name="gz::sim::systems::DiffDrive">
-      <left_joint>rear_left_wheel_joint</left_joint>
-      <right_joint>rear_right_wheel_joint</right_joint>
-      <wheel_separation>0.16</wheel_separation>
-      <wheel_radius>0.05</wheel_radius>
-      <max_linear_acceleration>1.0</max_linear_acceleration>
-      <max_angular_acceleration>2.0</max_angular_acceleration>
-      <topic>cmd_vel</topic>
-      <odom_topic>odom</odom_topic>
-      <tf_topic>tf</tf_topic>
-      <frame_id>odom</frame_id>
-      <child_frame_id>base_link</child_frame_id>
-      <odom_publish_frequency>50.0</odom_publish_frequency>
-    </plugin>
   </gazebo>
   <!-- All transmission blocks removed - ROS1 legacy, replaced by ros2_control -->
