Commit message: Colorize mechatrobot's model

File: mechatrobot/urdf/robot.urdf (robot description, URDF)
Before this commit: robot robot, 4 links, 3 joints
Links:
- added link range_sensor_left_transducer; visual cylinder length=0.012 radius=0.008
- added link range_sensor_right_transducer; visual cylinder length=0.012 radius=0.008
- link range_sensor: geometry visual box size=0.045 0.020 0.002
Joints:
- added joint sensor_to_left_transducer: type fixed, parent range_sensor, child range_sensor_left_transducer, origin xyz=0.006 0.0166 0 rpy=0 0 0
- added joint sensor_to_right_transducer: type fixed, parent range_sensor, child range_sensor_right_transducer, origin xyz=0.006 -0.0166 0 rpy=0 0 0

Commit message: Rename base_link to breadboard link

File: mechatrobot/urdf/robot.urdf (robot description, URDF)
Before this commit: robot robot, 6 links, 5 joints
Links:
- removed link base_link
- added link breadboard_link; visual box size=0.053 0.082 0.01
Joints:
- joint base_to_motor: parent base_link -> breadboard_link
- joint base_to_sensor: parent base_link -> breadboard_link

Commit message: Add arduino nano (seeeduino nano)

File: mechatrobot/urdf/robot.urdf (robot description, URDF)
Before this commit: robot robot, 6 links, 5 joints
Links:
- added link arduino_nano; visual box size=0.045 0.018 0.005
Joints:
- added joint breadboard_to_arduino: type fixed, parent breadboard_link, child arduino_nano, origin xyz=0 0.022 0.0075 rpy=0 0 1.57

Commit message: Add

File: mechatrobot/urdf/robot.urdf (robot description, URDF)
Before this commit: robot robot, 7 links, 6 joints
Links:
- added link led; visual cylinder length=0.002 radius=0.0025
Joints:
- added joint arduino_to_led: type fixed, parent arduino_nano, child led, origin xyz=0.01 0 0.0035 rpy=0 0 0
