Commit message: Add

File: mechatrobot_ros2/urdf/robot.urdf (robot description, URDF)
Before this commit: robot robot, 8 links, 7 joints
Links:
- added link base_link; visual box size=0.053 0.082 0.01
- link motor_link: geometry visual mesh filename=package://mechatrobot_ros2/urdf/28BYJ-48.STL scale=0.001 0.001 0.001
Joints:
- added joint base_to_breadboard: type fixed, parent base_link, child breadboard_link, origin xyz=0 0 0.005 rpy=0 0 0

Commit message: Add

File: mechatrobot_ros2/urdf/robot.urdf (robot description, URDF)
Before this commit: robot robot, 9 links, 8 joints
Joints:
- joint joint1: limit lower=-3.14 upper=3.14 effort=1000.0 velocity=0.5 -> lower=-3.14 upper=3.14 effort=1000.0 velocity=2.0
